File: Electronics/MainDisk/MainDisk.sch (KiCad schematic (older format))
At the start: 36 parts, among them J1 Conn_02x03_Odd_Even, Q1 Q_NPN_BEC, SW1 SW_Push, SW2 SW_SPST, U1 ATMEGA328PB-AURCT-ND, U2 TSOP4840-ND, Y1 535-10212-1-ND

Commit message: Continued work on the Disk
Parts:
- removed C5, C6: 1uF, Capacitor_SMD:C_0805_2012Metric, symbol Device:C_Small
- added D5, D6: LED, LED_SMD:LED_0805_2012Metric, symbol Device:LED
- added R4, R5: 470R, Resistor_SMD:R_0805_2012Metric, symbol Device:R_Small
- added R6, R8: 100k, Resistor_SMD:R_0805_2012Metric, symbol Device:R_Small
- added R7: 30k, Resistor_SMD:R_0805_2012Metric, symbol Device:R_Small
- added SW3: SW_Push, Button_Switch_SMD:SW_SPST_B3U-1000P, symbol Switch:SW_Push
- R3: value R_Small -> 470R
Connections:
- net +BATT: now also R4.1, R5.1, R6.2, R8.2
- net BAT_SENS: now also R6.1, R7.1
- net GND: now also R7.2, SW3.1
- net RESET: now also R8.1, SW3.2
- net at U1.13 (PB1): now also D5.1 (K)
- net at U1.14 (PB2): now also D6.1 (K)
- new net: D5.2 (A), R4.2
- new net: D6.2 (A), R5.2
Other:
- note added: "B_LOW"
- note added: "PWR\n"
- moved on the sheet: BZ1, SW1

Commit message: More smol tweaks to the bacon
Parts:
- J1: value Conn_02x03_Odd_Even -> 0015912060
Connections:
- net at U1.2 (PD4): no longer JP5.1 (A)
- net at U1.25 (PC2): now also JP2.1 (A)
- net at U1.26 (PC3): now also JP3.1 (A)
- net at U1.30 (PD0): now also JP4.1 (A); no longer JP2.1 (A)
- net at U1.31 (PD1): now also JP5.1 (A); no longer JP3.1 (A)
- net at U1.32 (PD2): now also JP6.1 (A); no longer JP4.1 (A)
- net at U1.9 (PD5): no longer JP6.1 (A)
Other:
- moved on the sheet: JP2, JP3, JP4, JP5, JP6
Changed lines of the file:
@@
 L Jumper:SolderJumper_2_Open JP2
 U 1 1 5CE382B3
+P 7225 4050
+F 0 "JP2" H 7500 4050 50  0000 C CNN
+F 1 "SolderJumper_2_Open" H 7225 4164 50  0001 C CNN
+F 2 "Jumper:SolderJumper-2_P1.3mm_Open_RoundedPad1.0x1.5mm" H 7225 4050 50  0001 C CNN
+F 3 "~" H 7225 4050 50  0001 C CNN
+	1    7225 4050
+	1    0    0    -1
+$EndComp
+$Comp
+L Jumper:SolderJumper_2_Open JP3
+U 1 1 5CE3854F
+P 7225 4150
+F 0 "JP3" H 7500 4150 50  0000 C CNN
+F 1 "SolderJumper_2_Open" H 7225 4264 50  0001 C CNN
+F 2 "Jumper:SolderJumper-2_P1.3mm_Open_RoundedPad1.0x1.5mm" H 7225 4150 50  0001 C CNN
+F 3 "~" H 7225 4150 50  0001 C CNN
+	1    7225 4150
+	1    0    0    -1
+$EndComp
+$Comp
+L Jumper:SolderJumper_2_Open JP4
+U 1 1 5CE385D8
 P 7225 4250
-F 0 "JP2" H 7500 4250 50  0000 C CNN
+F 0 "JP4" H 7500 4250 50  0000 C CNN
 F 1 "SolderJumper_2_Open" H 7225 4364 50  0001 C CNN
 F 2 "Jumper:SolderJumper-2_P1.3mm_Open_RoundedPad1.0x1.5mm" H 7225 4250 50  0001 C CNN
@@
 $EndComp
 $Comp
-L Jumper:SolderJumper_2_Open JP3
-U 1 1 5CE3854F
+L power:GND #PWR0118
+U 1 1 5CE39289
+P 7575 4150
+F 0 "#PWR0118" H 7575 3900 50  0001 C CNN
+F 1 "GND" V 7580 4022 50  0000 R CNN
+F 2 "" H 7575 4150 50  0001 C CNN
+F 3 "" H 7575 4150 50  0001 C CNN
+	1    7575 4150
+	0    -1   -1   0
+$EndComp
+Wire Wire Line
+	7375 4050 7400 4050
+Wire Wire Line
+	7400 4050 7400 4150
+Wire Wire Line
+	7400 4250 7375 4250
+Wire Wire Line
+	7375 4150 7400 4150
+Connection ~ 7400 4150
+Wire Wire Line
+	7400 4150 7400 4250
+Wire Wire Line
+	7400 4150 7575 4150
+$Comp
+L Jumper:SolderJumper_2_Open JP5
+U 1 1 5CE43B7B
 P 7225 4350
-F 0 "JP3" H 7500 4350 50  0000 C CNN
+F 0 "JP5" H 7500 4350 50  0000 C CNN
 F 1 "SolderJumper_2_Open" H 7225 4464 50  0001 C CNN
 F 2 "Jumper:SolderJumper-2_P1.3mm_Open_RoundedPad1.0x1.5mm" H 7225 4350 50  0001 C CNN
@@
 $EndComp
 $Comp
-L Jumper:SolderJumper_2_Open JP4
-U 1 1 5CE385D8
+L Jumper:SolderJumper_2_Open JP6
+U 1 1 5CE43C12
 P 7225 4450
-F 0 "JP4" H 7500 4450 50  0000 C CNN
+F 0 "JP6" H 7500 4450 50  0000 C CNN
 F 1 "SolderJumper_2_Open" H 7225 4564 50  0001 C CNN
 F 2 "Jumper:SolderJumper-2_P1.3mm_Open_RoundedPad1.0x1.5mm" H 7225 4450 50  0001 C CNN
@@
 	1    0    0    -1
 $EndComp
-$Comp
-L power:GND #PWR0118
-U 1 1 5CE39289
-P 7575 4350
-F 0 "#PWR0118" H 7575 4100 50  0001 C CNN
-F 1 "GND" V 7580 4222 50  0000 R CNN
-F 2 "" H 7575 4350 50  0001 C CNN
-F 3 "" H 7575 4350 50  0001 C CNN
-	1    7575 4350
-	0    -1   -1   0
-$EndComp
-Wire Wire Line
-	7375 4250 7400 4250
-Wire Wire Line
-	7400 4250 7400 4350
-Wire Wire Line
-	7400 4450 7375 4450
-Wire Wire Line
-	7375 4350 7400 4350
-Connection ~ 7400 4350
-Wire Wire Line
-	7400 4350 7400 4450
-Wire Wire Line
-	7400 4350 7575 4350
-Wire Wire Line
-	6425 4650 7075 4650
-Wire Wire Line
-	6425 4750 7075 4750
-$Comp
-L Jumper:SolderJumper_2_Open JP5
-U 1 1 5CE43B7B
-P 7225 4650
-F 0 "JP5" H 7500 4650 50  0000 C CNN
-F 1 "SolderJumper_2_Open" H 7225 4764 50  0001 C CNN
-F 2 "Jumper:SolderJumper-2_P1.3mm_Open_RoundedPad1.0x1.5mm" H 7225 4650 50  0001 C CNN
-F 3 "~" H 7225 4650 50  0001 C CNN
-	1    7225 4650
-	1    0    0    -1
-$EndComp
-$Comp
-L Jumper:SolderJumper_2_Open JP6
-U 1 1 5CE43C12
-P 7225 4750
-F 0 "JP6" H 7500 4750 50  0000 C CNN
-F 1 "SolderJumper_2_Open" H 7225 4864 50  0001 C CNN
-F 2 "Jumper:SolderJumper-2_P1.3mm_Open_RoundedPad1.0x1.5mm" H 7225 4750 50  0001 C CNN
-F 3 "~" H 7225 4750 50  0001 C CNN
-	1    7225 4750
-	1    0    0    -1
-$EndComp
-Wire Wire Line
-	7375 4650 7400 4650
-Wire Wire Line
-	7400 4650 7400 4450
-Connection ~ 7400 4450
-Wire Wire Line
-	7375 4750 7400 4750
-Wire Wire Line
-	7400 4750 7400 4650
-Connection ~ 7400 4650
+Wire Wire Line
+	7375 4450 7400 4450
+Wire Wire Line
+	7400 4450 7400 4350
+Connection ~ 7400 4250
 $Comp
 L power:GND #PWR0119
@@
 P 6275 1175
 F 0 "J1" H 6325 1492 50  0000 C CNN
-F 1 "Conn_02x03_Odd_Even" H 6325 1401 50  0000 C CNN
+F 1 "0015912060" H 6325 1401 50  0000 C CNN
 F 2 "Connector_PinHeader_2.54mm:PinHeader_2x03_P2.54mm_Vertical_SMD" H 6275 1175 50  0001 C CNN
 F 3 "~" H 6275 1175 50  0001 C CNN
@@
 Text Label 4125 2500 2    50   ~ 0
 BAT_SENS
+Wire Wire Line
+	7375 4350 7400 4350
+Connection ~ 7400 4350
+Wire Wire Line
+	7400 4350 7400 4250
+Wire Wire Line
+	6425 3650 7050 3650
+Wire Wire Line
+	7050 3650 7050 4050
+Wire Wire Line
+	7050 4050 7075 4050
+Wire Wire Line
+	7075 4150 7000 4150
+Wire Wire Line
+	7000 4150 7000 3750
+Wire Wire Line
+	7000 3750 6425 3750
 $EndSCHEMATC

Commit message: More or less Rev. 1
Parts:
- added J2: Conn_01x02_Male, Connector_PinHeader_2.00mm:PinHeader_1x02_P2.00mm_Vertical, symbol Connector:Conn_01x02_Male
Connections:
- net WS2812: now reaches U1.2 (PD4)
- net WS2812: now also D1.4 (DIN)
- net at D2.1 (K), Q1.3 (C): now also J2.2 (Pin_2)
- net at D2.2 (A), R1.2: now also J2.1 (Pin_1)
Other:
- moved on the sheet: C9, D2, Q1, R1, R2, R3, U2
Changed lines of the file:
@@
 L Device:Q_NPN_BEC Q1
 U 1 1 5CE084BB
-P 9375 5550
-F 0 "Q1" H 9566 5596 50  0000 L CNN
-F 1 "Q_NPN_BEC" H 9566 5505 50  0000 L CNN
-F 2 "Package_TO_SOT_SMD:SOT-23" H 9575 5650 50  0001 C CNN
-F 3 "~" H 9375 5550 50  0001 C CNN
-	1    9375 5550
+P 6050 6950
+F 0 "Q1" H 6241 6996 50  0000 L CNN
+F 1 "Q_NPN_BEC" H 6241 6905 50  0000 L CNN
+F 2 "Package_TO_SOT_SMD:SOT-23" H 6250 7050 50  0001 C CNN
+F 3 "~" H 6050 6950 50  0001 C CNN
+	1    6050 6950
 	1    0    0    -1
 $EndComp
@@
 L Device:LED_ALT D2
 U 1 1 5CE08853
-P 9475 5150
-F 0 "D2" V 9513 5032 50  0000 R CNN
-F 1 "475-2866-1-ND" V 9422 5032 50  0000 R CNN
-F 2 "LED_SMD:LED_PLCC-2" H 9475 5150 50  0001 C CNN
-F 3 "~" H 9475 5150 50  0001 C CNN
-	1    9475 5150
+P 6150 6550
+F 0 "D2" V 6188 6432 50  0000 R CNN
+F 1 "475-2866-1-ND" V 6097 6432 50  0000 R CNN
+F 2 "LED_SMD:LED_PLCC-2" H 6150 6550 50  0001 C CNN
+F 3 "~" H 6150 6550 50  0001 C CNN
+	1    6150 6550
 	0    -1   -1   0
 $EndComp
@@
 L power:GND #PWR0110
 U 1 1 5CE1B578
-P 9475 5750
-F 0 "#PWR0110" H 9475 5500 50  0001 C CNN
-F 1 "GND" H 9480 5577 50  0000 C CNN
-F 2 "" H 9475 5750 50  0001 C CNN
-F 3 "" H 9475 5750 50  0001 C CNN
-	1    9475 5750
-	1    0    0    -1
-$EndComp
-Wire Wire Line
-	9475 5300 9475 5350
+P 6150 7150
+F 0 "#PWR0110" H 6150 6900 50  0001 C CNN
+F 1 "GND" H 6155 6977 50  0000 C CNN
+F 2 "" H 6150 7150 50  0001 C CNN
+F 3 "" H 6150 7150 50  0001 C CNN
+	1    6150 7150
+	1    0    0    -1
+$EndComp
+Wire Wire Line
+	6150 6700 6150 6725
 $Comp
 L Device:R_Small R1
 U 1 1 5CE1C283
-P 9475 4900
-F 0 "R1" H 9534 4946 50  0000 L CNN
-F 1 "49R" H 9534 4855 50  0000 L CNN
-F 2 "Resistor_SMD:R_0805_2012Metric" H 9475 4900 50  0001 C CNN
-F 3 "~" H 9475 4900 50  0001 C CNN
-	1    9475 4900
+P 6150 6250
+F 0 "R1" H 6209 6296 50  0000 L CNN
+F 1 "49R" H 6209 6205 50  0000 L CNN
+F 2 "Resistor_SMD:R_0805_2012Metric" H 6150 6250 50  0001 C CNN
+F 3 "~" H 6150 6250 50  0001 C CNN
+	1    6150 6250
 	1    0    0    -1
 $EndComp
@@
 L power:+BATT #PWR0111
 U 1 1 5CE1C46E
-P 9475 4800
-F 0 "#PWR0111" H 9475 4650 50  0001 C CNN
-F 1 "+BATT" H 9490 4973 50  0000 C CNN
-F 2 "" H 9475 4800 50  0001 C CNN
-F 3 "" H 9475 4800 50  0001 C CNN
-	1    9475 4800
+P 6150 6125
+F 0 "#PWR0111" H 6150 5975 50  0001 C CNN
+F 1 "+BATT" H 6165 6298 50  0000 C CNN
+F 2 "" H 6150 6125 50  0001 C CNN
+F 3 "" H 6150 6125 50  0001 C CNN
+	1    6150 6125
 	1    0    0    -1
 $EndComp
@@
 L Interface_Optical:TSOP41xx U2
 U 1 1 5CE288EB
-P 7550 5675
-F 0 "U2" V 7491 5963 50  0000 L CNN
-F 1 "TSOP4840-ND" V 7582 5963 50  0000 L CNN
-F 2 "OptoDevice:Vishay_MOLD-3Pin" H 7500 5300 50  0001 C CNN
-F 3 "http://www.vishay.com/docs/82460/tsop45.pdf" H 8200 5975 50  0001 C CNN
-	1    7550 5675
+P 4550 6550
+F 0 "U2" V 3975 6300 50  0000 L CNN
+F 1 "TSOP4840-ND" V 4050 6300 50  0000 L CNN
+F 2 "OptoDevice:Vishay_MOLD-3Pin" H 4500 6175 50  0001 C CNN
+F 3 "http://www.vishay.com/docs/82460/tsop45.pdf" H 5200 6850 50  0001 C CNN
+	1    4550 6550
 	0    1    1    0
 $EndComp
@@
 L power:GND #PWR0119
 U 1 1 5CE4A9E3
-P 7350 6125
-F 0 "#PWR0119" H 7350 5875 50  0001 C CNN
-F 1 "GND" H 7355 5952 50  0000 C CNN
-F 2 "" H 7350 6125 50  0001 C CNN
-F 3 "" H 7350 6125 50  0001 C CNN
-	1    7350 6125
+P 4350 7000
+F 0 "#PWR0119" H 4350 6750 50  0001 C CNN
+F 1 "GND" H 4355 6827 50  0000 C CNN
+F 2 "" H 4350 7000 50  0001 C CNN
+F 3 "" H 4350 7000 50  0001 C CNN
+	1    4350 7000
 	1    0    0    -1
 $EndComp
@@
 L Device:C_Small C9
 U 1 1 5CE4B4B8
-P 7875 6200
-F 0 "C9" H 7967 6246 50  0000 L CNN
-F 1 "1uF" H 7967 6155 50  0000 L CNN
-F 2 "Capacitor_SMD:C_0805_2012Metric" H 7875 6200 50  0001 C CNN
-F 3 "~" H 7875 6200 50  0001 C CNN
-	1    7875 6200
-	1    0    0    -1
-$EndComp
-Wire Wire Line
-	7750 6075 7875 6075
-Wire Wire Line
-	7875 6075 7875 6100
+P 4875 7075
+F 0 "C9" H 4967 7121 50  0000 L CNN
+F 1 "1uF" H 4967 7030 50  0000 L CNN
+F 2 "Capacitor_SMD:C_0805_2012Metric" H 4875 7075 50  0001 C CNN
+F 3 "~" H 4875 7075 50  0001 C CNN
+	1    4875 7075
+	1    0    0    -1
+$EndComp
+Wire Wire Line
+	4750 6950 4875 6950
+Wire Wire Line
+	4875 6950 4875 6975
 $Comp
 L power:GND #PWR0120
 U 1 1 5CE4D6FF
-P 7875 6300
-F 0 "#PWR0120" H 7875 6050 50  0001 C CNN
-F 1 "GND" H 7880 6127 50  0000 C CNN
-F 2 "" H 7875 6300 50  0001 C CNN
-F 3 "" H 7875 6300 50  0001 C CNN
-	1    7875 6300
+P 4875 7175
+F 0 "#PWR0120" H 4875 6925 50  0001 C CNN
+F 1 "GND" H 4880 7002 50  0000 C CNN
+F 2 "" H 4875 7175 50  0001 C CNN
+F 3 "" H 4875 7175 50  0001 C CNN
+	1    4875 7175
 	1    0    0    -1
 $EndComp
@@
 L Device:R_Small R2
 U 1 1 5CE4D9BC
-P 8175 6075
-F 0 "R2" V 7979 6075 50  0000 C CNN
-F 1 "100R" V 8070 6075 50  0000 C CNN
-F 2 "Resistor_SMD:R_0805_2012Metric" H 8175 6075 50  0001 C CNN
-F 3 "~" H 8175 6075 50  0001 C CNN
-	1    8175 6075
+P 5150 6950
+F 0 "R2" V 4954 6950 50  0000 C CNN
+F 1 "100R" V 5045 6950 50  0000 C CNN
+F 2 "Resistor_SMD:R_0805_2012Metric" H 5150 6950 50  0001 C CNN
+F 3 "~" H 5150 6950 50  0001 C CNN
+	1    5150 6950
 	0    1    1    0
 $EndComp
 Wire Wire Line
-	7875 6075 8075 6075
-Connection ~ 7875 6075
+	4875 6950 5050 6950
+Connection ~ 4875 6950
 $Comp
 L power:+BATT #PWR0121
 U 1 1 5CE4FEBD
-P 8450 6075
-F 0 "#PWR0121" H 8450 5925 50  0001 C CNN
-F 1 "+BATT" V 8465 6203 50  0000 L CNN
-F 2 "" H 8450 6075 50  0001 C CNN
-F 3 "" H 8450 6075 50  0001 C CNN
-	1    8450 6075
-	0    1    1    0
-$EndComp
-Wire Wire Line
-	8275 6075 8450 6075
-Wire Wire Line
-	7350 6125 7350 6075
-Wire Wire Line
-	7550 6075 7550 6350
-Text Label 7550 6350 1    50   ~ 0
+P 5325 6950
+F 0 "#PWR0121" H 5325 6800 50  0001 C CNN
+F 1 "+BATT" V 5340 7078 50  0000 L CNN
+F 2 "" H 5325 6950 50  0001 C CNN
+F 3 "" H 5325 6950 50  0001 C CNN
+	1    5325 6950
+	1    0    0    -1
+$EndComp
+Wire Wire Line
+	5250 6950 5325 6950
+Wire Wire Line
+	4350 7000 4350 6950
+Wire Wire Line
+	4550 6950 4550 7225
+Text Label 4550 7225 1    50   ~ 0
 IR_IN
 $Comp
@@
 L Device:R_Small R3
 U 1 1 5CE5B147
-P 9075 5550
-F 0 "R3" V 8879 5550 50  0000 C CNN
-F 1 "470R" V 8970 5550 50  0000 C CNN
-F 2 "Resistor_SMD:R_0805_2012Metric" H 9075 5550 50  0001 C CNN
-F 3 "~" H 9075 5550 50  0001 C CNN
-	1    9075 5550
+P 5750 6950
+F 0 "R3" V 5554 6950 50  0000 C CNN
+F 1 "470R" V 5645 6950 50  0000 C CNN
+F 2 "Resistor_SMD:R_0805_2012Metric" H 5750 6950 50  0001 C CNN
+F 3 "~" H 5750 6950 50  0001 C CNN
+	1    5750 6950
 	0    1    1    0
 $EndComp
-Wire Wire Line
-	8975 5550 8625 5550
-Text Label 8625 5550 0    50   ~ 0
+Text Label 5525 6950 1    50   ~ 0
 IR_LED
 Wire Wire Line
@@
 Wire Wire Line
 	7000 3750 6425 3750
+Wire Wire Line
+	5650 6950 5525 6950
+$Comp
+L Connector:Conn_01x02_Male J2
+U 1 1 5CE77F3B
+P 5700 6500
+F 0 "J2" H 5806 6678 50  0000 C CNN
+F 1 "Conn_01x02_Male" H 5806 6587 50  0000 C CNN
+F 2 "Connector_PinHeader_2.00mm:PinHeader_1x02_P2.00mm_Vertical" H 5700 6500 50  0001 C CNN
+F 3 "~" H 5700 6500 50  0001 C CNN
+	1    5700 6500
+	1    0    0    -1
+$EndComp
+Wire Wire Line
+	6150 6125 6150 6150
+Wire Wire Line
+	6150 6350 6150 6375
+Wire Wire Line
+	5900 6500 5900 6375
+Wire Wire Line
+	5900 6375 6150 6375
+Connection ~ 6150 6375
+Wire Wire Line
+	6150 6375 6150 6400
+Wire Wire Line
+	6150 6725 5900 6725
+Wire Wire Line
+	5900 6725 5900 6600
+Connection ~ 6150 6725
+Wire Wire Line
+	6150 6725 6150 6750
+Wire Wire Line
+	6425 4650 6775 4650
+Text Label 6775 4650 2    50   ~ 0
+WS2812
+Text Label 7700 2925 0    50   ~ 0
+WS2812
+Wire Wire Line
+	8050 2925 7700 2925
 $EndSCHEMATC
