File: Electronics/MainDisk/MainDisk.kicad_pcb (KiCad board)
At the start: 2 copper layers, 37.8 x 37.8 mm, 43 parts, among them J1 0015912060, J2 Conn_01x02_Male, Q1 Q_NPN_BEC, SW1 SW_Push, SW2 SW_SPST, SW3 SW_Push, U1 ATMEGA328PB-AURCT-ND, U2 TSOP4840-ND, Y1 535-10212-1-ND

Commit message: Add changes to KiCAD PCB
Other:
- outline, holes or cut-outs redrawn
Changed lines of the file:
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@@
   (general
     (thickness 1.6)
-    (drawings 28)
+    (drawings 30)
     (tracks 294)
     (zones 0)
@@
     (zone_45_only no)
     (trace_min 0.2)
-    (segment_width 0.6)
+    (segment_width 0.2)
     (edge_width 0.2)
     (via_size 0.8)
@@
     )
   )
-  (gr_line (start 140.9319 84.8995) (end 141.1986 85.0519) (layer Edge.Cuts) (width 0.2))
+  (gr_circle (center 152.4 69.85) (end 142.1892 85.7758) (layer Edge.Cuts) (width 0.2))
+  (gr_line (start 141.1986 85.0519) (end 140.91412 84.87664) (layer Eco2.User) (width 0.2))
+  (gr_line (start 144.399 86.995) (end 144.6911 87.122) (layer Eco2.User) (width 0.2))
   (gr_text A1 (at 152.146 84.328 90) (layer B.Mask)
     (effects (font (size 1 1) (thickness 0.18)) (justify mirror))
@@
     (effects (font (size 1 1) (thickness 0.15)))
   )
-  (gr_arc (start 152.4 69.85) (end 144.399 86.995) (angle -347.7085751) (layer Edge.Cuts) (width 0.2))
-  (gr_arc (start 142.748 86.106) (end 144.399 86.995) (angle -174.0722099) (layer Edge.Cuts) (width 0.2))
+  (gr_arc (start 152.4 69.85) (end 144.6911 87.122) (angle -346.7) (layer Eco2.User) (width 0.2))
+  (gr_arc (start 142.748 86.106) (end 144.399 86.995) (angle -174.1) (layer Eco2.User) (width 0.2))
   (gr_circle (center 152.4 69.85) (end 170.9 69.85) (layer F.SilkS) (width 0.5))
   (gr_circle (center 153.035 58.293) (end 157.539474 58.293) (layer B.SilkS) (width 0.2))
